Commit message: Update paths for Allegro hand
Signed-off-by: Eric Heiden <eric-heiden@outlook.com>

File: wonik_allegro/urdf/allegro_hand_description_left.urdf (robot description, URDF)
Before this commit: robot allegro_hand_left, 21 links, 20 joints
Links:
- link link_0.0: geometry collision box size=0.0196 0.0275 0.0164; visual mesh filename=package://wonik_allegro/meshes/link_0.0.STL
- link link_1.0: geometry collision box size=0.0196 0.0275 0.054; visual mesh filename=package://wonik_allegro/meshes/link_1.0.STL
- link link_10.0: geometry collision box size=0.0196 0.0275 0.0384; visual mesh filename=package://wonik_allegro/meshes/link_2.0.STL
- link link_11.0: geometry collision box size=0.0196 0.0275 0.0267; visual mesh filename=package://wonik_allegro/meshes/link_3.0.STL
- link link_11.0_tip: geometry collision sphere radius=0.012; visual mesh filename=package://wonik_allegro/meshes/link_3.0_tip.STL
- link link_12.0: geometry collision box size=0.0358 0.034 0.0455; visual mesh filename=package://wonik_allegro/meshes/link_12.0_left.STL
- link link_13.0: geometry collision box size=0.0196 0.0275 0.0177; visual mesh filename=package://wonik_allegro/meshes/link_13.0.STL
- link link_14.0: geometry collision box size=0.0196 0.0275 0.0514; visual mesh filename=package://wonik_allegro/meshes/link_14.0.STL
- link link_15.0: geometry collision box size=0.0196 0.0275 0.0423; visual mesh filename=package://wonik_allegro/meshes/link_15.0.STL
- link link_15.0_tip: geometry collision sphere radius=0.012; visual mesh filename=package://wonik_allegro/meshes/link_15.0_tip.STL
- link link_2.0: geometry collision box size=0.0196 0.0275 0.0384; visual mesh filename=package://wonik_allegro/meshes/link_2.0.STL
- link link_3.0: geometry collision box size=0.0196 0.0275 0.0267; visual mesh filename=package://wonik_allegro/meshes/link_3.0.STL
- link link_3.0_tip: geometry collision sphere radius=0.012; visual mesh filename=package://wonik_allegro/meshes/link_3.0_tip.STL
- link link_4.0: geometry collision box size=0.0196 0.0275 0.0164; visual mesh filename=package://wonik_allegro/meshes/link_0.0.STL
- link link_5.0: geometry collision box size=0.0196 0.0275 0.054; visual mesh filename=package://wonik_allegro/meshes/link_1.0.STL
- link link_6.0: geometry collision box size=0.0196 0.0275 0.0384; visual mesh filename=package://wonik_allegro/meshes/link_2.0.STL
- link link_7.0: geometry collision box size=0.0196 0.0275 0.0267; visual mesh filename=package://wonik_allegro/meshes/link_3.0.STL
- link link_7.0_tip: geometry collision sphere radius=0.012; visual mesh filename=package://wonik_allegro/meshes/link_3.0_tip.STL
- link link_8.0: geometry collision box size=0.0196 0.0275 0.0164; visual mesh filename=package://wonik_allegro/meshes/link_0.0.STL
- link link_9.0: geometry collision box size=0.0196 0.0275 0.054; visual mesh filename=package://wonik_allegro/meshes/link_1.0.STL
- link palm_link: geometry collision box size=0.0408 0.1130 0.095; visual mesh filename=package://wonik_allegro/meshes/base_link_left.STL

File: wonik_allegro/urdf/allegro_hand_description_right.urdf (robot description, URDF)
Before this commit: robot allegro_hand_right, 21 links, 20 joints
Links:
- link link_0.0: geometry collision box size=0.0196 0.0275 0.0164; visual mesh filename=package://wonik_allegro/meshes/link_0.0.STL
- link link_1.0: geometry collision box size=0.0196 0.0275 0.054; visual mesh filename=package://wonik_allegro/meshes/link_1.0.STL
- link link_10.0: geometry collision box size=0.0196 0.0275 0.0384; visual mesh filename=package://wonik_allegro/meshes/link_2.0.STL
- link link_11.0: geometry collision box size=0.0196 0.0275 0.0267; visual mesh filename=package://wonik_allegro/meshes/link_3.0.STL
- link link_11.0_tip: geometry collision sphere radius=0.012; visual mesh filename=package://wonik_allegro/meshes/link_3.0_tip.STL
- link link_12.0: geometry collision box size=0.0358 0.034 0.0455; visual mesh filename=package://wonik_allegro/meshes/link_12.0_right.STL
- link link_13.0: geometry collision box size=0.0196 0.0275 0.0177; visual mesh filename=package://wonik_allegro/meshes/link_13.0.STL
- link link_14.0: geometry collision box size=0.0196 0.0275 0.0514; visual mesh filename=package://wonik_allegro/meshes/link_14.0.STL
- link link_15.0: geometry collision box size=0.0196 0.0275 0.0423; visual mesh filename=package://wonik_allegro/meshes/link_15.0.STL
- link link_15.0_tip: geometry collision sphere radius=0.012; visual mesh filename=package://wonik_allegro/meshes/link_15.0_tip.STL
- link link_2.0: geometry collision box size=0.0196 0.0275 0.0384; visual mesh filename=package://wonik_allegro/meshes/link_2.0.STL
- link link_3.0: geometry collision box size=0.0196 0.0275 0.0267; visual mesh filename=package://wonik_allegro/meshes/link_3.0.STL
- link link_3.0_tip: geometry collision sphere radius=0.012; visual mesh filename=package://wonik_allegro/meshes/link_3.0_tip.STL
- link link_4.0: geometry collision box size=0.0196 0.0275 0.0164; visual mesh filename=package://wonik_allegro/meshes/link_0.0.STL
- link link_5.0: geometry collision box size=0.0196 0.0275 0.054; visual mesh filename=package://wonik_allegro/meshes/link_1.0.STL
- link link_6.0: geometry collision box size=0.0196 0.0275 0.0384; visual mesh filename=package://wonik_allegro/meshes/link_2.0.STL
- link link_7.0: geometry collision box size=0.0196 0.0275 0.0267; visual mesh filename=package://wonik_allegro/meshes/link_3.0.STL
- link link_7.0_tip: geometry collision sphere radius=0.012; visual mesh filename=package://wonik_allegro/meshes/link_3.0_tip.STL
- link link_8.0: geometry collision box size=0.0196 0.0275 0.0164; visual mesh filename=package://wonik_allegro/meshes/link_0.0.STL
- link link_9.0: geometry collision box size=0.0196 0.0275 0.054; visual mesh filename=package://wonik_allegro/meshes/link_1.0.STL
- link palm_link: geometry collision box size=0.0408 0.1130 0.095; visual mesh filename=package://wonik_allegro/meshes/base_link.STL
